Commit message: Four joint manipulator added for inverse kinematics example.

File: models/urdf/two_link_2.xacro (robot description, xacro)
@@ -95,9 +95,18 @@
   <!-- Joint between the first link and the new link -->
   <joint name="${box_name}/link_joint1" type="revolute">
-    <origin xyz="0.0 -0.075 0.0" rpy="0 0 0" />
+    <origin xyz="0.2 -0.075 -0.07" rpy="0 0 0" />
     <parent link="${box_name}/box" />
     <child link="${box_name}/arm1" />
     <axis xyz="0 1 0" />
-    <limit lower="${-pi}" upper="${pi}" effort="10.01" velocity="1.01" />
+    <limit lower="${-pi}" upper="${pi}" effort="50.01" velocity="1.01" />
+    <dynamics damping="0.0" friction="0.1"/>
+  </joint>
+  <!-- Joint between the first link and the new link -->
+  <joint name="${box_name}/link_joint11" type="revolute">
+    <origin xyz="0.225 -0.05 0.0" rpy="0 0 0" />
+    <parent link="${box_name}/arm1" />
+    <child link="${box_name}/arm11" />
+    <axis xyz="0 1 0" />
+    <limit lower="${-pi}" upper="${pi}" effort="50.01" velocity="1.01" />
     <dynamics damping="0.0" friction="0.1"/>
   </joint>
@@ -108,9 +117,9 @@
     <!-- Joint between the first link and the new link -->
   <joint name="${box_name}/link_joint2" type="revolute">
-    <origin xyz="0.0 0.075 0.0" rpy="0 0 0" />
+    <origin xyz="0.2 0.075 -0.07" rpy="0 0 0" />
     <parent link="${box_name}/box" />
     <child link="${box_name}/arm2" />
     <axis xyz="0 1 0" />
-    <limit lower="${-pi}" upper="${pi}" effort="10.01" velocity="1.01" />
+    <limit lower="${-pi}" upper="${pi}" effort="50.01" velocity="1.01" />
     <dynamics damping="0.0" friction="0.1"/>
   </joint>
@@ -125,8 +134,8 @@
     </hardware>
     <joint name="${box_name}/link_joint1">
-      <param name="pos_kp">20</param>
+      <param name="pos_kp">4</param>
       <param name="pos_ki">1</param>
-      <param name="pos_kd">10</param>
-      <param name="pos_max_integral_error">10</param>
+      <param name="pos_kd">1</param>
+      <param name="pos_max_integral_error">1</param>
       <command_interface name="position_pid"/>
       <state_interface name="position"/>
@@ -135,8 +144,8 @@
     </joint>
     <joint name="${box_name}/link_joint2">
-      <param name="pos_kp">20</param>
+      <param name="pos_kp">4</param>
       <param name="pos_ki">1</param>
-      <param name="pos_kd">10</param>
-      <param name="pos_max_integral_error">10</param>
+      <param name="pos_kd">1</param>
+      <param name="pos_max_integral_error">1</param>
       <command_interface name="position_pid"/>
       <state_interface name="position"/>

Commit message: Four joint manipulator added for inverse kinematics example.

File: models/urdf/two_link_2.xacro (robot description, xacro)
@@ -95,16 +95,7 @@
   <!-- Joint between the first link and the new link -->
   <joint name="${box_name}/link_joint1" type="revolute">
-    <origin xyz="0.2 -0.075 -0.07" rpy="0 0 0" />
+    <origin xyz="0.0 -0.075 -0.00" rpy="0 0 0" />
     <parent link="${box_name}/box" />
     <child link="${box_name}/arm1" />
-    <axis xyz="0 1 0" />
-    <limit lower="${-pi}" upper="${pi}" effort="50.01" velocity="1.01" />
-    <dynamics damping="0.0" friction="0.1"/>
-  </joint>
-  <!-- Joint between the first link and the new link -->
-  <joint name="${box_name}/link_joint11" type="revolute">
-    <origin xyz="0.225 -0.05 0.0" rpy="0 0 0" />
-    <parent link="${box_name}/arm1" />
-    <child link="${box_name}/arm11" />
     <axis xyz="0 1 0" />
     <limit lower="${-pi}" upper="${pi}" effort="50.01" velocity="1.01" />
@@ -117,5 +108,5 @@
     <!-- Joint between the first link and the new link -->
   <joint name="${box_name}/link_joint2" type="revolute">
-    <origin xyz="0.2 0.075 -0.07" rpy="0 0 0" />
+    <origin xyz="0.0 0.075 -0.0" rpy="0 0 0" />
     <parent link="${box_name}/box" />
     <child link="${box_name}/arm2" />
