Commit message: A joint commander for simple leg is added.

File: models/urdf/dog_quadruped3.xacro (robot description, xacro)
@@ -113,5 +113,5 @@
       <!-- ab/ad around X -->
       <axis xyz="0 0 1"/>
-      <limit lower="-1.5" upper="1.5" effort="500" velocity="6.0"/>
+      <limit lower="${-pi}" upper="${pi}" effort="500" velocity="6.0"/>
       <dynamics damping="0.5" friction="0.01"/>
     </joint>
@@ -136,5 +136,5 @@
       <!-- ab/ad around X -->
       <axis xyz="0 1 0"/>
-      <limit lower="-2.0" upper="2.0" effort="50" velocity="6.0"/>
+      <limit lower="${-pi}" upper="${pi}" effort="50" velocity="6.0"/>
       <dynamics damping="0.5" friction="0.01"/>
     </joint>
@@ -178,5 +178,5 @@
       <!-- ab/ad around X -->
       <axis xyz="0 1 0"/>
-      <limit lower="-2.0" upper="2.0" effort="50" velocity="6.0"/>
+      <limit lower="${-pi}" upper="${pi}" effort="50" velocity="6.0"/>
       <dynamics damping="0.5" friction="0.01"/>
     </joint>

File: models/urdf/simpleLeg.xacro (robot description, xacro)
@@ -91,4 +91,9 @@
     <xacro:inertial_box m="10" x="0.1" y="0.1" z="0.5"/>
   </link>
+  <gazebo reference="pillar">
+    <material>Gazebo/Grey</material>
+      <mu1>150.01</mu1>
+      <mu2>150.01</mu2>
+  </gazebo>
   <joint name="platform_to_pillar" type="fixed">
     <parent link="platform"/>
@@ -145,5 +150,5 @@
       <!-- ab/ad around X -->
       <axis xyz="0 0 1"/>
-      <limit lower="-1.5" upper="1.5" effort="50" velocity="6.0"/>
+      <limit lower="${-pi}" upper="${pi}" effort="50" velocity="6.0"/>
       <dynamics damping="0.5" friction="0.01"/>
     </joint>
@@ -168,5 +173,5 @@
       <!-- ab/ad around X -->
       <axis xyz="0 1 0"/>
-      <limit lower="-2.0" upper="2.0" effort="50" velocity="6.0"/>
+      <limit lower="${-pi}" upper="${pi}" effort="50" velocity="6.0"/>
       <dynamics damping="0.5" friction="0.01"/>
     </joint>
@@ -210,5 +215,5 @@
       <!-- ab/ad around X -->
       <axis xyz="0 1 0"/>
-      <limit lower="-2.0" upper="2.0" effort="50" velocity="6.0"/>
+      <limit lower="${-pi}" upper="${pi}" effort="50" velocity="6.0"/>
       <dynamics damping="0.5" friction="0.01"/>
     </joint>
